Commit message: MSA용 urdf업로드

File: kat_description/urdf_moveit/open_manipulator_x_moveit.urdf (robot description, URDF)
Before this commit: robot open_manipulator_x, 8 links, 7 joints
Links:
- link end_effector_link: geometry collision box size=0.01 0.01 0.01; visual box size=0.01 0.01 0.01
- link gripper_left_link: mass 1.0e-03 -> 0.001
- link gripper_right_link: mass 1.0e-03 -> 0.001
Joints:
- joint end_effector_joint: origin xyz=0.126 0.0 0.0 rpy=0 0 0 -> xyz=0.126 0 0 rpy=0 0 0
- joint gripper_left_joint: origin xyz=0.0817 0.021 0.0 rpy=0 0 0 -> xyz=0.0817 0.021 0 rpy=0 0 0
- joint joint1: limit lower=-3.141592653589793 upper=3.141592653589793 effort=1000 velocity=4.8 -> lower=-3.14159265 upper=3.14159265 effort=1000 velocity=4.8; origin xyz=0.012 0.0 0.0 rpy=0 0 0 -> xyz=0.012 0 0 rpy=0 0 0
- joint joint2: origin xyz=0.0 0.0 0.0595 rpy=0 0 0 -> xyz=0 0 0.0595 rpy=0 0 0
- joint joint4: origin xyz=0.124 0.0 0.0 rpy=0 0 0 -> xyz=0.124 0 0 rpy=0 0 0
