Commit message: 종강 이후 수정

File: kat_description/urdf/assembled/omx_board_assenbled.urdf (robot description, URDF)
Before this commit: robot open_manipulator_x, 9 links, 8 joints
Links:
- link board_link: geometry collision mesh filename=package://kat_description/meshes/board/board_with_marker.stl scale=0.001 0.001 0.001; visual mesh filename=package://kat_description/meshes/board/board_with_marker.stl scale=0.001 0.001 0.001

File: kat_description/urdf/open_manipulator_x/open_manipulator_x.urdf.xacro (robot description, xacro)
@@ -1,5 +1,5 @@
 <?xml version="1.0"?>
 <robot name="open_manipulator_x" xmlns:xacro="http://ros.org/wiki/xacro">
-  <xacro:arg name="prefix" default="omx_" />
+  <xacro:arg name="prefix" default="" />
   <xacro:arg name="use_sim" default="false" />
   <xacro:arg name="use_fake_hardware" default="false" />
@@ -7,5 +7,5 @@
   <xacro:arg name="port_name" default="/dev/ttyUSB0" />
   <xacro:arg name="ros2_control_type" default="open_manipulator_x" />
-  <xacro:include filename="$(find kat_description)/gazebo/open_manipulator_x.gazebo.xacro" />
+  <xacro:include filename="$(find kat_sim)/gazebo/open_manipulator_x/open_manipulator_x.gazebo.xacro" />
   <xacro:include filename="$(find kat_description)/urdf/open_manipulator_x/open_manipulator_x_arm.urdf.xacro" />
   <xacro:include filename="$(find kat_control)/ros2_control/$(arg ros2_control_type).ros2_control.xacro" />
@@ -25,5 +25,5 @@
   <gazebo>
     <plugin filename="gz_ros2_control-system" name="gz_ros2_control::GazeboSimROS2ControlPlugin">
-      <parameters>$(find kat_bringup)/config/open_manipulator_x/hardware_controller_manager.yaml</parameters>
+      <parameters>$(find kat_control)/config/open_manipulator_x/hardware_controller_manager.yaml</parameters>
     </plugin>
   </gazebo>

File: kat_description/urdf/open_manipulator_x/open_manipulator_x_arm.urdf.xacro (robot description, xacro)
@@ -189,5 +189,5 @@
       </inertial>
     </link>
-    <joint name="${prefix}gripper_right_joint" type="prismatic">
+    <joint name="${prefix}gripper_right_joint_mimic" type="prismatic">
       <parent link="${prefix}link5"/>
       <child link="${prefix}gripper_right_link"/>

File: kat_moveit_config/config/open_manipulator_x.ros2_control.xacro (robot description, xacro)
@@ -36,11 +36,4 @@
                 <state_interface name="velocity"/>
             </joint>
-            <joint name="gripper_left_joint">
-                <command_interface name="position"/>
-                <state_interface name="position">
-                  <param name="initial_value">${initial_positions['gripper_left_joint']}</param>
-                </state_interface>
-                <state_interface name="velocity"/>
-            </joint>
         </ros2_control>
     </xacro:macro>

File: kat_moveit_config/config/open_manipulator_x.urdf.xacro (robot description, xacro)
@@ -3,5 +3,5 @@
     <xacro:arg name="initial_positions_file" default="initial_positions.yaml" />
     <!-- Import open_manipulator_x urdf file -->
-    <xacro:include filename="$(find kat_description)/urdf/moveit_setup_assistant/open_manipulator_x_moveit.urdf" />
+    <xacro:include filename="$(find kat_description)/urdf/open_manipulator_x/open_manipulator_x_msa.urdf.xacro" />
     <!-- Import control_xacro -->
     <xacro:include filename="open_manipulator_x.ros2_control.xacro" />
