Commit message: 실제 하드웨어 연결 수정

File: kat_control/ros2_control/open_manipulator_x.ros2_control.xacro (robot description, xacro)
@@ -1,6 +1,10 @@
 <?xml version="1.0"?>
 <robot xmlns:xacro="http://www.ros.org/wiki/xacro">
-  <xacro:macro name="open_manipulator_x_system" params="name prefix port_name:=^|/dev/ttyUSB0 use_sim:=^|false use_fake_hardware:=^|false fake_sensor_commands:=^|false">
+  <xacro:macro name="open_manipulator_x_system"
+    params="name prefix port_name:=^|/dev/ttyUSB0 use_sim:=^|false use_fake_hardware:=^|false fake_sensor_commands:=^|false">
     <ros2_control name="${name}" type="system">
+      <!-- ===================== -->
+      <!-- Hardware definition -->
+      <!-- ===================== -->
       <xacro:if value="$(arg use_sim)">
         <hardware>
@@ -43,4 +47,5 @@
             <param name="reboot_dxl_srv_name">dynamixel_hardware_interface/reboot_dxl</param>
             <param name="set_dxl_torque_srv_name">dynamixel_hardware_interface/set_dxl_torque</param>
+            <!-- Gripper mapping -->
             <param name="use_revolute_to_prismatic_gripper">1</param>
             <param name="revolute_to_prismatic_dxl">dxl5</param>
@@ -53,4 +58,7 @@
         </hardware>
       </xacro:unless>
+      <!-- ===================== -->
+      <!-- Joint interfaces -->
+      <!-- ===================== -->
       <joint name="${prefix}joint1">
         <command_interface name="position"/>
@@ -83,13 +91,7 @@
         <state_interface name="effort"/>
       </joint>
-      <xacro:if value="$(arg use_sim)">
-        <joint name="${prefix}gripper_right_joint">
-          <param name="mimic">${prefix}gripper_left_joint</param>
-          <param name="multiplier">1</param>
-          <state_interface name="position"/>
-          <state_interface name="velocity"/>
-          <state_interface name="effort"/>
-        </joint>
-      </xacro:if>
+      <!-- ===================== -->
+      <!-- Dynamixel GPIO (XL430 safe: NO Drive Mode write) -->
+      <!-- ===================== -->
       <gpio name="dxl1">
         <param name="type">dxl</param>
@@ -97,6 +99,4 @@
         <command_interface name="Goal Position"/>
         <state_interface name="Present Position"/>
-        <state_interface name="Present Velocity"/>
-        <state_interface name="Present Current"/>
         <param name="Operating Mode">3</param>
         <param name="Position P Gain">800</param>
@@ -105,5 +105,4 @@
         <param name="Profile Velocity">20</param>
         <param name="Profile Acceleration">10</param>
-        <param name="Drive Mode">4</param>
         <param name="Return Delay Time">0</param>
       </gpio>
@@ -113,6 +112,4 @@
         <command_interface name="Goal Position"/>
         <state_interface name="Present Position"/>
-        <state_interface name="Present Velocity"/>
-        <state_interface name="Present Current"/>
         <param name="Operating Mode">3</param>
         <param name="Position P Gain">800</param>
@@ -121,5 +118,4 @@
         <param name="Profile Velocity">20</param>
         <param name="Profile Acceleration">10</param>
-        <param name="Drive Mode">4</param>
         <param name="Return Delay Time">0</param>
       </gpio>
@@ -129,6 +125,4 @@
         <command_interface name="Goal Position"/>
         <state_interface name="Present Position"/>
-        <state_interface name="Present Velocity"/>
-        <state_interface name="Present Current"/>
         <param name="Operating Mode">3</param>
         <param name="Position P Gain">800</param>
@@ -137,5 +131,4 @@
         <param name="Profile Velocity">20</param>
         <param name="Profile Acceleration">10</param>
-        <param name="Drive Mode">4</param>
         <param name="Return Delay Time">0</param>
       </gpio>
@@ -145,6 +138,4 @@
         <command_interface name="Goal Position"/>
         <state_interface name="Present Position"/>
-        <state_interface name="Present Velocity"/>
-        <state_interface name="Present Current"/>
         <param name="Operating Mode">3</param>
         <param name="Position P Gain">800</param>
@@ -153,7 +144,7 @@
         <param name="Profile Velocity">20</param>
         <param name="Profile Acceleration">10</param>
-        <param name="Drive Mode">4</param>
         <param name="Return Delay Time">0</param>
       </gpio>
+      <!-- Gripper motor: XL430 safe -->
       <gpio name="dxl5">
         <param name="type">dxl</param>
@@ -161,12 +152,8 @@
         <command_interface name="Goal Position"/>
         <state_interface name="Present Position"/>
-        <state_interface name="Present Velocity"/>
-        <state_interface name="Present Current"/>
-        <param name="Operating Mode">5</param>
+        <param name="Operating Mode">3</param>
         <param name="Profile Velocity">20</param>
         <param name="Profile Acceleration">10</param>
-        <param name="Drive Mode">4</param>
         <param name="Return Delay Time">0</param>
-        <param name="Goal Current">200</param>
       </gpio>
     </ros2_control>
