Commit message: 주석제거 및 joint2 허용범위 확대

File: open_manipulator_x/kat_description/urdf/open_manipulator_x/open_manipulator_x_arm.urdf.xacro (robot description, xacro)
@@ -66,5 +66,5 @@
       <origin xyz="0.0 0.0 0.0595" rpy="0 0 0"/>
       <axis xyz="0 1 0"/>
-      <limit velocity="4.8" effort="1000" lower="${-1.5}" upper="${1.5}" />
+      <limit velocity="4.8" effort="1000" lower="${-2.0}" upper="${2.0}" />
       <dynamics damping="0.1"/>
     </joint>

Commit message: 20260108 수정

File: open_manipulator_x/kat_description/urdf/open_manipulator_x/open_manipulator_x_arm.urdf.xacro (robot description, xacro)
@@ -15,10 +15,10 @@
         </material>
       </visual>
-      <collision>
+      <!-- <collision>
         <origin xyz="0 0 0" rpy="0 0 0"/>
         <geometry>
           <mesh filename="${meshes_file_direction}/link1.stl" scale="0.001 0.001 0.001"/>
         </geometry>
-      </collision>
+      </collision> -->
        <inertial>
         <origin xyz="3.0876154e-04 0.0000000e+00 -1.2176461e-04" />
@@ -79,10 +79,10 @@
         </material>
       </visual>
-      <collision>
+      <!-- <collision>
         <origin xyz="0 0 0" rpy="0 0 0"/>
         <geometry>
           <mesh filename="${meshes_file_direction}/link3.stl" scale="0.001 0.001 0.001"/>
         </geometry>
-      </collision>
+      </collision> -->
        <inertial>
         <origin xyz="1.0308393e-02 3.7743363e-04 1.0170197e-01" />

File: open_manipulator_x/kat_sim/gazebo/open_manipulator_x/open_manipulator_x.gazebo.xacro (robot description, xacro)
@@ -33,10 +33,10 @@
   <gazebo reference="${prefix}end_effector_link">
   </gazebo>
-  <xacro:SimpleTransmission trans="${prefix}trans1" joint="${prefix}joint1" actuator="${prefix}actuator1" />
+  <!-- <xacro:SimpleTransmission trans="${prefix}trans1" joint="${prefix}joint1" actuator="${prefix}actuator1" />
   <xacro:SimpleTransmission trans="${prefix}trans2" joint="${prefix}joint2" actuator="${prefix}actuator2" />
   <xacro:SimpleTransmission trans="${prefix}trans3" joint="${prefix}joint3" actuator="${prefix}actuator3" />
   <xacro:SimpleTransmission trans="${prefix}trans4" joint="${prefix}joint4" actuator="${prefix}actuator4" />
   <xacro:SimpleTransmission trans="${prefix}trans5" joint="${prefix}gripper_left_joint" actuator="${prefix}actuator5" />
-  <xacro:SimpleTransmission trans="${prefix}trans6" joint="${prefix}gripper_right_joint" actuator="${prefix}actuator6" />
+  <xacro:SimpleTransmission trans="${prefix}trans6" joint="${prefix}gripper_right_joint" actuator="${prefix}actuator6" /> -->
   </xacro:macro>
 </robot>

Commit message: 20260112

File: open_manipulator_x/kat_description/urdf/open_manipulator_x/open_manipulator_x_arm.urdf.xacro (robot description, xacro)
@@ -175,10 +175,10 @@
         </material>
       </visual>
-      <collision>
+      <!-- <collision>
         <origin xyz="0 0 0" rpy="0 0 0"/>
         <geometry>
           <mesh filename="${meshes_file_direction}/gripper_left_palm.stl" scale="0.001 0.001 0.001"/>
         </geometry>
-      </collision>
+      </collision> -->
       <inertial>
         <origin xyz="0 0 0" />
@@ -208,10 +208,10 @@
         </material>
       </visual>
-      <collision>
+      <!-- <collision>
         <origin xyz="0 0 0" rpy="0 0 0"/>
         <geometry>
           <mesh filename="${meshes_file_direction}/gripper_right_palm.stl" scale="0.001 0.001 0.001"/>
         </geometry>
-      </collision>
+      </collision> -->
       <inertial>
         <origin xyz="0 0 0" />

Commit message: 20260114 양은서 수정: kat_control 컴퓨터 이동 리스너 수정

File: open_manipulator_x/kat_description/urdf/open_manipulator_x/open_manipulator_x_arm.urdf.xacro (robot description, xacro)
@@ -47,10 +47,10 @@
         </material>
       </visual>
-      <collision>
+      <!-- <collision>
         <origin xyz="0 0 0.019" rpy="0 0 0"/>
         <geometry>
           <mesh filename="${meshes_file_direction}/link2.stl" scale="0.001 0.001 0.001"/>
         </geometry>
-      </collision>
+      </collision> -->
        <inertial>
         <origin xyz="-3.0184870e-04 5.4043684e-04 ${0.018 + 2.9433464e-02}" />
